Commit message: Use existing macro instead of copy.
Signed-off-by: Jelmer de Wolde <jelmer.de.wolde@alliander.com>

File: rcdt_mobile_manipulator/config/franka.urdf.xacro (robot description, xacro)
@@ -4,8 +4,11 @@
 SPDX-License-Identifier: Apache-2.0
 -->
-<robot xmlns:xacro="http://www.ros.org/wiki/xacro" name="franka">
-  <!-- Define arm: -->
-  <xacro:arg name="arm_id" default="fr3" />
-  <xacro:arg name="ee_id" default="franka_hand" />
+<robot xmlns:xacro="http://www.ros.org/wiki/xacro"
+  name="franka">
+  <!-- Define arm and end-effector: -->
+  <xacro:arg name="arm_id"
+    default="fr3" />
+  <xacro:arg name="ee_id"
+    default="franka_hand" />
   <!-- Load arm: -->
   <xacro:include filename="$(find franka_description)/robots/common/franka_robot.xacro" />
@@ -19,30 +22,9 @@
     gazebo="true"
     xyz="0 0 0.32" />
-  <!-- Based on franka_arm.ros2_control.xacro: -->
-  <!-- Load ros2 control but use general ign_ros2_control, instead of franka_ign_ros_control: -->
-  <ros2_control name="FrankaHardwareInterface" type="system" namespace="franka">
-    <hardware>
-      <plugin>ign_ros2_control/IgnitionSystem</plugin>
-    </hardware>
-    <xacro:macro name="configure_joint" params="joint_name initial_position">
-      <joint name="${joint_name}">
-        <command_interface name="velocity" />
-        <command_interface name="position" />
-        <state_interface name="position">
-          <param name="initial_value">${initial_position}</param>
-        </state_interface>
-        <state_interface name="velocity" />
-        <param name="initial_value">0.0</param>
-        <state_interface name="effort" />
-      </joint>
-    </xacro:macro>
-    <xacro:configure_joint joint_name="$(arg arm_id)_joint1" initial_position="0.0" />
-    <xacro:configure_joint joint_name="$(arg arm_id)_joint2" initial_position="${-pi/4}" />
-    <xacro:configure_joint joint_name="$(arg arm_id)_joint3" initial_position="0.0" />
-    <xacro:configure_joint joint_name="$(arg arm_id)_joint4" initial_position="${-3*pi/4}" />
-    <xacro:configure_joint joint_name="$(arg arm_id)_joint5" initial_position="0.0" />
-    <xacro:configure_joint joint_name="$(arg arm_id)_joint6" initial_position="${pi/2}" />
-    <xacro:configure_joint joint_name="$(arg arm_id)_joint7" initial_position="${pi/4}" />
-    <xacro:configure_joint joint_name="$(arg arm_id)_finger_joint1" initial_position="0.0" />
-  </ros2_control>
+  <!-- Load ros2 control: -->
+  <xacro:include filename="$(find franka_description)/robots/common/franka_arm.ros2_control.xacro" />
+  <xacro:franka_arm_ros2_control arm_id="$(arg arm_id)"
+    robot_ip=""
+    hand="true"
+    ign_ros2_control="true" />
 </robot>
